File: v2/_autosave-v2.kicad_sch (KiCad schematic)
At the start: 103 parts, among them SW1 SW_Push, SW10 SW_Push, SW11 SW_Push, SW12 SW_Push, SW13 SW_Push, SW14 SW_Push, SW15 SW_Push, SW16 SW_Push, SW17 SW_Push, SW18 SW_Push, SW19 SW_Push, SW2 SW_Push, SW20 SW_Push, SW21 SW_Push, SW22 SW_Push, SW23 SW_Push, SW24 SW_Push, SW25 SW_Push, SW26 SW_Push, SW27 SW_Push, SW28 SW_Push, SW29 SW_Push, SW3 SW_Push, SW30 SW_Push, SW31 SW_Push, SW32 SW_Push, SW4 SW_Push, SW5 SW_Push, SW6 SW_Push, SW7 SW_Push, SW8 SW_Push, SW9 SW_Push, U1 Pico

Commit message: did some layout using a plugin
Parts:
- removed D36, D41, D47, D53, D59, D65: SK6812MINI, reversible-kicad-footprints:MX-1U-SK6812Mini-E, symbol LED:SK6812MINI
- renumbered D11 to D10, D16 to D11, D21 to D12, D26 to D13, D30 to D14, D3 to D15, D7 to D16, D12 to D17, D17 to D18, D22 to D19, D5 to D2, D27 to D20, D31 to D21, D4 to D22, D8 to D23, D13 to D24, D18 to D25, D23 to D26, D28 to D27, D70 to D28, D9 to D29, D10 to D3, D14 to D30, D19 to D31, D24 to D32, D15 to D4, D20 to D5, D25 to D6, D29 to D7, D2 to D8, D6 to D9, D32 to LED1, D56 to LED10, D50 to LED11, D44 to LED12, D38 to LED13, D33 to LED14, D34 to LED15, D39 to LED16, D45 to LED17, D51 to LED18, D57 to LED19, D37 to LED2, D63 to LED20, D68 to LED21, D69 to LED22, D64 to LED23, D58 to LED24, D52 to LED25, D46 to LED26, D40 to LED27, D35 to LED28, D42 to LED29, D43 to LED3, D48 to LED30, D54 to LED31, D60 to LED32, D49 to LED4, D55 to LED5, D61 to LED6, D66 to LED7, D67 to LED8, D62 to LED9, SW11 to SW10, SW16 to SW11, SW21 to SW12, SW26 to SW13, SW30 to SW14, SW3 to SW15, SW7 to SW16, SW12 to SW17, SW17 to SW18, SW22 to SW19, SW5 to SW2, SW27 to SW20, SW31 to SW21, SW4 to SW22, SW8 to SW23, SW13 to SW24, SW18 to SW25, SW23 to SW26, SW28 to SW27, SW32 to SW28, SW9 to SW29, SW10 to SW3, SW14 to SW30, SW19 to SW31, SW24 to SW32, SW15 to SW4, SW20 to SW5, SW25 to SW6, SW29 to SW7, SW2 to SW8, SW6 to SW9
Connections:
- net at LED22.1 (DOUT): now also LED29.3 (DIN)
- net at LED31.3 (DIN): no longer LED30.1 (DOUT)
- net at LED29.1 (DOUT): no longer LED30.3 (DIN)
Other:
- moved on the sheet: LED29, LED30, LED31, LED32
