File: v2/_autosave-v2.kicad_sch (KiCad schematic)
At the start: 105 parts, among them J1 Conn_01x04_Pin, J2 Conn_01x04_Pin, J3 Conn_01x04_Pin, SW1 SW_Push, SW10 SW_Push, SW11 SW_Push, SW12 SW_Push, SW13 SW_Push, SW14 SW_Push, SW15 SW_Push, SW16 SW_Push, SW17 SW_Push, SW18 SW_Push, SW19 SW_Push, SW2 SW_Push, SW20 SW_Push, SW21 SW_Push, SW22 SW_Push, SW23 SW_Push, SW24 SW_Push, SW25 SW_Push, SW26 SW_Push, SW27 SW_Push, SW28 SW_Push, SW29 SW_Push, SW3 SW_Push, SW30 SW_Push, SW31 SW_Push, SW32 SW_Push, SW33 RotaryEncoder_Switch, SW4 SW_Push, SW5 SW_Push, SW6 SW_Push, SW7 SW_Push, SW8 SW_Push, SW9 SW_Push, U1 Pico, U2 Pico

Commit message: I screwed up some layout
Parts:
- D1, D10, D11, D12, D13, D14, D15, D16, D17, D18, D19, D2, D20, D21, D22, D23, D24, D25, D26, D27, D28, D29, D3, D30, D31, D32, D33, D4, D5, D6, D7, D8, D9: footprint Diode_THT:D_5W_P10.16mm_Horizontal -> Keebio-Parts:Diode-Hybrid-Back
Changed lines of the file:
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@@
 			)
 		)
-		(property "Footprint" "Diode_THT:D_5W_P10.16mm_Horizontal"
+		(property "Footprint" "Keebio-Parts:Diode-Hybrid-Back"
 			(at 265.43 85.09 0)
 			(effects
@@
 			)
 		)
-		(property "Footprint" "Diode_THT:D_5W_P10.16mm_Horizontal"
+		(property "Footprint" "Keebio-Parts:Diode-Hybrid-Back"
 			(at 227.33 85.09 0)
 			(effects
@@
 			)
 		)
-		(property "Footprint" "Diode_THT:D_5W_P10.16mm_Horizontal"
+		(property "Footprint" "Keebio-Parts:Diode-Hybrid-Back"
 			(at 151.13 44.45 0)
 			(effects
@@
 			)
 		)
-		(property "Footprint" "Diode_THT:D_5W_P10.16mm_Horizontal"
+		(property "Footprint" "Keebio-Parts:Diode-Hybrid-Back"
 			(at 208.28 44.45 0)
 			(effects
@@
 			)
 		)
-		(property "Footprint" "Diode_THT:D_5W_P10.16mm_Horizontal"
+		(property "Footprint" "Keebio-Parts:Diode-Hybrid-Back"
 			(at 246.38 125.73 0)
 			(effects
@@
 			)
 		)
-		(property "Footprint" "Diode_THT:D_5W_P10.16mm_Horizontal"
+		(property "Footprint" "Keebio-Parts:Diode-Hybrid-Back"
 			(at 227.33 105.41 0)
 			(effects
@@
 			)
 		)
-		(property "Footprint" "Diode_THT:D_5W_P10.16mm_Horizontal"
+		(property "Footprint" "Keebio-Parts:Diode-Hybrid-Back"
 			(at 151.13 105.41 0)
 			(effects
@@
 			)
 		)
-		(property "Footprint" "Diode_THT:D_5W_P10.16mm_Horizontal"
+		(property "Footprint" "Keebio-Parts:Diode-Hybrid-Back"
 			(at 246.38 85.09 0)
 			(effects
@@
 			)
 		)
-		(property "Footprint" "Diode_THT:D_5W_P10.16mm_Horizontal"
+		(property "Footprint" "Keebio-Parts:Diode-Hybrid-Back"
 			(at 171.45 64.77 0)
 			(effects
@@
 			)
 		)
-		(property "Footprint" "Diode_THT:D_5W_P10.16mm_Horizontal"
+		(property "Footprint" "Keebio-Parts:Diode-Hybrid-Back"
 			(at 189.23 125.73 0)
 			(effects
@@
 			)
 		)
-		(property "Footprint" "Diode_THT:D_5W_P10.16mm_Horizontal"
+		(property "Footprint" "Keebio-Parts:Diode-Hybrid-Back"
 			(at 265.43 44.45 0)
 			(effects
@@
 			)
 		)
-		(property "Footprint" "Diode_THT:D_5W_P10.16mm_Horizontal"
+		(property "Footprint" "Keebio-Parts:Diode-Hybrid-Back"
 			(at 208.28 64.77 0)
 			(effects
@@
 			)
 		)
-		(property "Footprint" "Diode_THT:D_5W_P10.16mm_Horizontal"
+		(property "Footprint" "Keebio-Parts:Diode-Hybrid-Back"
 			(at 189.23 85.09 0)
 			(effects
@@
 			)
 		)
-		(property "Footprint" "Diode_THT:D_5W_P10.16mm_Horizontal"
+		(property "Footprint" "Keebio-Parts:Diode-Hybrid-Back"
 			(at 265.43 105.41 0)
 			(effects
@@
 			)
 		)
-		(property "Footprint" "Diode_THT:D_5W_P10.16mm_Horizontal"
+		(property "Footprint" "Keebio-Parts:Diode-Hybrid-Back"
 			(at 189.23 64.77 0)
 			(effects
@@
 			)
 		)
-		(property "Footprint" "Diode_THT:D_5W_P10.16mm_Horizontal"
+		(property "Footprint" "Keebio-Parts:Diode-Hybrid-Back"
 			(at 208.28 85.09 0)
 			(effects
@@
 			)
 		)
-		(property "Footprint" "Diode_THT:D_5W_P10.16mm_Horizontal"
+		(property "Footprint" "Keebio-Parts:Diode-Hybrid-Back"
 			(at 246.38 64.77 0)
 			(effects
@@
 			)
 		)
-		(property "Footprint" "Diode_THT:D_5W_P10.16mm_Horizontal"
+		(property "Footprint" "Keebio-Parts:Diode-Hybrid-Back"
 			(at 208.28 125.73 0)
 			(effects
@@
 			)
 		)
-		(property "Footprint" "Diode_THT:D_5W_P10.16mm_Horizontal"
+		(property "Footprint" "Keebio-Parts:Diode-Hybrid-Back"
 			(at 208.28 105.41 0)
 			(effects
@@
 			)
 		)
-		(property "Footprint" "Diode_THT:D_5W_P10.16mm_Horizontal"
+		(property "Footprint" "Keebio-Parts:Diode-Hybrid-Back"
 			(at 171.45 44.45 0)
 			(effects
@@
 			)
 		)
-		(property "Footprint" "Diode_THT:D_5W_P10.16mm_Horizontal"
+		(property "Footprint" "Keebio-Parts:Diode-Hybrid-Back"
 			(at 227.33 44.45 0)
 			(effects
@@
 			)
 		)
-		(property "Footprint" "Diode_THT:D_5W_P10.16mm_Horizontal"
+		(property "Footprint" "Keebio-Parts:Diode-Hybrid-Back"
 			(at 246.38 105.41 0)
 			(effects
@@
 			)
 		)
-		(property "Footprint" "Diode_THT:D_5W_P10.16mm_Horizontal"
+		(property "Footprint" "Keebio-Parts:Diode-Hybrid-Back"
 			(at 227.33 64.77 0)
 			(effects
@@
 			)
 		)
-		(property "Footprint" "Diode_THT:D_5W_P10.16mm_Horizontal"
+		(property "Footprint" "Keebio-Parts:Diode-Hybrid-Back"
 			(at 227.33 125.73 0)
 			(effects
@@
 			)
 		)
-		(property "Footprint" "Diode_THT:D_5W_P10.16mm_Horizontal"
+		(property "Footprint" "Keebio-Parts:Diode-Hybrid-Back"
 			(at 171.45 125.73 0)
 			(effects
@@
 			)
 		)
-		(property "Footprint" "Diode_THT:D_5W_P10.16mm_Horizontal"
+		(property "Footprint" "Keebio-Parts:Diode-Hybrid-Back"
 			(at 151.13 85.09 0)
 			(effects
@@
 			)
 		)
-		(property "Footprint" "Diode_THT:D_5W_P10.16mm_Horizontal"
+		(property "Footprint" "Keebio-Parts:Diode-Hybrid-Back"
 			(at 151.13 64.77 0)
 			(effects
@@
 			)
 		)
-		(property "Footprint" "Diode_THT:D_5W_P10.16mm_Horizontal"
+		(property "Footprint" "Keebio-Parts:Diode-Hybrid-Back"
 			(at 171.45 85.09 0)
 			(effects
@@
 			)
 		)
-		(property "Footprint" "Diode_THT:D_5W_P10.16mm_Horizontal"
+		(property "Footprint" "Keebio-Parts:Diode-Hybrid-Back"
 			(at 189.23 44.45 0)
 			(effects
@@
 			)
 		)
-		(property "Footprint" "Diode_THT:D_5W_P10.16mm_Horizontal"
+		(property "Footprint" "Keebio-Parts:Diode-Hybrid-Back"
 			(at 265.43 64.77 0)
 			(effects
@@
 			)
 		)
-		(property "Footprint" "Diode_THT:D_5W_P10.16mm_Horizontal"
+		(property "Footprint" "Keebio-Parts:Diode-Hybrid-Back"
 			(at 189.23 105.41 0)
 			(effects
@@
 			)
 		)
-		(property "Footprint" "Diode_THT:D_5W_P10.16mm_Horizontal"
+		(property "Footprint" "Keebio-Parts:Diode-Hybrid-Back"
 			(at 246.38 44.45 0)
 			(effects
@@
 			)
 		)
-		(property "Footprint" "Diode_THT:D_5W_P10.16mm_Horizontal"
+		(property "Footprint" "Keebio-Parts:Diode-Hybrid-Back"
 			(at 171.45 105.41 0)
 			(effects
