File: v2/v2.kicad_sch (KiCad schematic)
At the start: 103 parts, among them SW1 SW_Push, SW10 SW_Push, SW11 SW_Push, SW12 SW_Push, SW13 SW_Push, SW14 SW_Push, SW15 SW_Push, SW16 SW_Push, SW17 SW_Push, SW18 SW_Push, SW19 SW_Push, SW2 SW_Push, SW20 SW_Push, SW21 SW_Push, SW22 SW_Push, SW23 SW_Push, SW24 SW_Push, SW25 SW_Push, SW26 SW_Push, SW27 SW_Push, SW28 SW_Push, SW29 SW_Push, SW3 SW_Push, SW30 SW_Push, SW31 SW_Push, SW32 SW_Push, SW4 SW_Push, SW5 SW_Push, SW6 SW_Push, SW7 SW_Push, SW8 SW_Push, SW9 SW_Push, U1 Pico

Commit message: schematic finished + some pcb
Parts:
- removed D36, D41, D47, D53, D59, D65: SK6812MINI, reversible-kicad-footprints:MX-1U-SK6812Mini-E, symbol LED:SK6812MINI
- added D33: D, Diode_THT:D_5W_P10.16mm_Horizontal, symbol Device:D
- added J1, J2: Conn_01x04_Pin, Keebio-Parts:I2C_Breakout, symbol Connector:Conn_01x04_Pin
- added J3: Conn_01x04_Pin, Keebio-Parts:TRRS-PJ-320A-dual, symbol Connector:Conn_01x04_Pin
- added R1, R2: 5K, Keebio-Parts:Resistor, symbol Device:R
- added R3: 5K (LEFT), Keebio-Parts:Resistor, symbol Device:R
- added R4: 5K (RIGHT), Keebio-Parts:Resistor, symbol Device:R
- added SW33: RotaryEncoder_Switch, Keebio-Parts:RotaryEncoder_EC11, symbol Device:RotaryEncoder_Switch
- added U2: Pico, Module:RaspberryPi_Pico_SMD_HandSolder, symbol RPi_Pico:Pico
- U1: footprint RPi_Pico:RPi_Pico_SMD_TH -> Module:RaspberryPi_Pico_SMD_HandSolder
- renumbered D11 to D10, D16 to D11, D21 to D12, D26 to D13, D30 to D14, D3 to D15, D7 to D16, D12 to D17, D17 to D18, D22 to D19, D5 to D2, D27 to D20, D31 to D21, D4 to D22, D8 to D23, D13 to D24, D18 to D25, D23 to D26, D28 to D27, D70 to D28, D9 to D29, D10 to D3, D14 to D30, D19 to D31, D24 to D32, D15 to D4, D20 to D5, D25 to D6, D29 to D7, D2 to D8, D6 to D9, D32 to LED1, D56 to LED10, D50 to LED11, D44 to LED12, D38 to LED13, D33 to LED14, D34 to LED15, D39 to LED16, D45 to LED17, D51 to LED18, D57 to LED19, D37 to LED2, D63 to LED20, D68 to LED21, D69 to LED22, D64 to LED23, D58 to LED24, D52 to LED25, D46 to LED26, D40 to LED27, D35 to LED28, D42 to LED29, D43 to LED3, D48 to LED30, D54 to LED31, D60 to LED32, D49 to LED4, D55 to LED5, D61 to LED6, D66 to LED7, D67 to LED8, D62 to LED9, SW11 to SW10, SW16 to SW11, SW21 to SW12, SW26 to SW13, SW30 to SW14, SW3 to SW15, SW7 to SW16, SW12 to SW17, SW17 to SW18, SW22 to SW19, SW5 to SW2, SW27 to SW20, SW31 to SW21, SW4 to SW22, SW8 to SW23, SW13 to SW24, SW18 to SW25, SW23 to SW26, SW28 to SW27, SW32 to SW28, SW9 to SW29, SW10 to SW3, SW14 to SW30, SW19 to SW31, SW24 to SW32, SW15 to SW4, SW20 to SW5, SW25 to SW6, SW29 to SW7, SW2 to SW8, SW6 to SW9
Connections:
- net Col 1: now also U1.1 (GPIO0), U2.1 (GPIO0)
- net Col 2: now also U1.2 (GPIO1), U2.2 (GPIO1)
- net Col 3: now also U1.4 (GPIO2), U2.4 (GPIO2)
- net Col 4: now also U1.5 (GPIO3), U2.5 (GPIO3)
- net Col 5: now also U1.6 (GPIO4), U2.6 (GPIO4)
- net Col 6: now also U1.7 (GPIO5), SW33.S1, U2.7 (GPIO5)
- net Col 7: now also U1.9 (GPIO6), U2.9 (GPIO6)
- net GND: now also J1.1 (Pin_1), J2.1 (Pin_1), J3.1 (Pin_1), R4.2, SW33.C, U2.18 (GND), U2.23 (GND), U2.28 (GND), U2.3 (GND), U2.33 (AGND), U2.38 (GND), U2.42 (GND), U2.8 (GND); no longer U1.41 (SWCLK)
- net Row 1: now also U1.10 (GPIO7), U2.10 (GPIO7)
- net Row 2: now also U1.11 (GPIO8), U2.11 (GPIO8)
- net Row 3: now also U1.12 (GPIO9), U2.12 (GPIO9)
- net Row 4: now also U1.13 (GND), U2.13 (GND)
- net VBUS: now also J3.4 (Pin_4), U2.40 (VBUS)
- net SK6912PWM: now reaches LED1.3 (DIN)
- net at LED22.1 (DOUT): now also LED29.3 (DIN)
- net Row 5: now reaches D29.1 (K), D30.1 (K), D31.1 (K), D32.1 (K)
- net Row 5: now also U1.14 (GPIO10), D33.1 (K), U2.14 (GPIO10)
- net at LED31.3 (DIN): no longer LED30.1 (DOUT)
- net SPLIT SELECT: now reaches U1.21 (GPIO16)
- net SPLIT SELECT: now also R3.2, R4.1, U2.21 (GPIO16)
- net SERIAL B: now reaches U1.24 (GPIO18)
- net SERIAL B: now also J3.2 (Pin_2)
- net SERIAL A: now reaches U1.25 (GPIO19)
- net SERIAL A: now also J3.3 (Pin_3)
- net VSYS: now reaches U1.39 (VSYS)
- net VSYS: now also U2.39 (VSYS)
- net at LED29.1 (DOUT): no longer LED30.3 (DIN)
- new net +3.3V: J1.2 (Pin_2), J2.2 (Pin_2), R1.1, R2.2, R3.1, U2.36 (3V3)
- new net ENC A: R1.2, SW33.A
- new net ENC B: R2.1, SW33.B
- new net ENCSWB: D33.2 (A), SW33.S2
- new net SCA: J1.4 (Pin_4), J2.4 (Pin_4)
- new net SCL: J1.3 (Pin_3), J2.3 (Pin_3)
- new net SDA: U2.26 (GPIO20)
- new net SDL: U2.27 (GPIO21)
Other:
- note added: "Encoder"
- note added: "LED Matrix"
- note added: "OLED"
- note added: "Orhpeus Pico Bottom"
- note added: "Orhpeus Pico Top"
- note added: "Split Selector"
- note removed: "Orhpeus Pico"
- moved on the sheet: LED29, LED30, LED31, LED32
