File: v2/v2.kicad_pcb (KiCad board)
At the start: 2 copper layers, 178.7 x 150.8 mm, 119 parts, among them J2 Conn_01x04_Pin, J3 Conn_01x04_Pin, SW1 SW_Push, SW10 SW_Push, SW11 SW_Push, SW12 SW_Push, SW13 SW_Push, SW14 SW_Push, SW15 SW_Push, SW16 SW_Push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

Commit message: added qmk powered logo
Parts:
- added G***: LOGO, footprints:QMK_PoweredBy, F.Cu at (152.0, 195.5)
- added G***: LOGO, footprints:QMK_PoweredBy, B.Cu at (152.0, 195.5)
